File: Gate Inputs.sch (KiCad schematic (older format))
At the start: 37 parts, among them J10 WQP-PJ301M-12_JACK, J11 WQP-PJ301M-12_JACK, J12 WQP-PJ301M-12_JACK, J7 WQP-PJ301M-12_JACK, J8 WQP-PJ301M-12_JACK, J9 WQP-PJ301M-12_JACK, Q2 MMBT3904, Q3 MMBT3904, Q4 MMBT3904, Q5 MMBT3904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

Commit message: Rough Placement Completed
Completed the rough placement of the components on the pcb
Parts:
- D9: footprint Diode_SMD:D_SOT-23_NKA -> Package_TO_SOT_SMD:SOT-23
Changed lines of the file:
@@
 F 0 "D9" V 2146 5388 50  0000 L CNN
 F 1 "BAT54S" V 2055 5388 50  0000 L CNN
-F 2 "Diode_SMD:D_SOT-23_NKA" H 2175 5425 50  0001 L CNN
+F 2 "Package_TO_SOT_SMD:SOT-23" H 2175 5425 50  0001 L CNN
 F 3 "https://www.diodes.com/assets/Datasheets/ds11005.pdf" H 1980 5300 50  0001 C CNN
 	1    2100 5300

Commit message: Progress on routing tracks
Most of the power tracks are routed
Parts:
- R60, R61, R62, R63, R64, R65, R66, R67, R68, R69, R70, R71, R72, R73, R74, R75, R76, R77: footprint Resistor_SMD:R_0603_1608Metric_Pad1.05x0.95mm_HandSolder -> Resistor_SMD:R_0805_2012Metric
Changed lines of the file:
@@
 F 0 "R69" H 3132 2104 50  0000 R CNN
 F 1 "100k" H 3132 2195 50  0000 R CNN
-F 2 "Resistor_SMD:R_0603_1608Metric_Pad1.05x0.95mm_HandSolder" V 3240 2140 50  0001 C CNN
+F 2 "Resistor_SMD:R_0805_2012Metric" V 3240 2140 50  0001 C CNN
 F 3 "~" H 3200 2150 50  0001 C CNN
 	1    3200 2150
@@
 F 0 "R66" V 2705 1900 50  0000 C CNN
 F 1 "100k" V 2614 1900 50  0000 C CNN
-F 2 "Resistor_SMD:R_0603_1608Metric_Pad1.05x0.95mm_HandSolder" V 2540 1890 50  0001 C CNN
+F 2 "Resistor_SMD:R_0805_2012Metric" V 2540 1890 50  0001 C CNN
 F 3 "~" H 2500 1900 50  0001 C CNN
 	1    2500 1900
@@
 F 0 "R65" H 2318 2296 50  0000 L CNN
 F 1 "10k" H 2318 2205 50  0000 L CNN
-F 2 "Resistor_SMD:R_0603_1608Metric_Pad1.05x0.95mm_HandSolder" V 2290 2240 50  0001 C CNN
+F 2 "Resistor_SMD:R_0805_2012Metric" V 2290 2240 50  0001 C CNN
 F 3 "~" H 2250 2250 50  0001 C CNN
 	1    2250 2250
@@
 F 0 "R73" H 3132 3604 50  0000 R CNN
 F 1 "100k" H 3132 3695 50  0000 R CNN
-F 2 "Resistor_SMD:R_0603_1608Metric_Pad1.05x0.95mm_HandSolder" V 3240 3640 50  0001 C CNN
+F 2 "Resistor_SMD:R_0805_2012Metric" V 3240 3640 50  0001 C CNN
 F 3 "~" H 3200 3650 50  0001 C CNN
 	1    3200 3650
@@
 F 0 "R77" V 2705 3400 50  0000 C CNN
 F 1 "100k" V 2614 3400 50  0000 C CNN
-F 2 "Resistor_SMD:R_0603_1608Metric_Pad1.05x0.95mm_HandSolder" V 2540 3390 50  0001 C CNN
+F 2 "Resistor_SMD:R_0805_2012Metric" V 2540 3390 50  0001 C CNN
 F 3 "~" H 2500 3400 50  0001 C CNN
 	1    2500 3400
@@
 F 0 "R62" H 2318 3796 50  0000 L CNN
 F 1 "10k" H 2318 3705 50  0000 L CNN
-F 2 "Resistor_SMD:R_0603_1608Metric_Pad1.05x0.95mm_HandSolder" V 2290 3740 50  0001 C CNN
+F 2 "Resistor_SMD:R_0805_2012Metric" V 2290 3740 50  0001 C CNN
 F 3 "~" H 2250 3750 50  0001 C CNN
 	1    2250 3750
@@
 F 0 "R71" H 6632 2104 50  0000 R CNN
 F 1 "100k" H 6632 2195 50  0000 R CNN
-F 2 "Resistor_SMD:R_0603_1608Metric_Pad1.05x0.95mm_HandSolder" V 6740 2140 50  0001 C CNN
+F 2 "Resistor_SMD:R_0805_2012Metric" V 6740 2140 50  0001 C CNN
 F 3 "~" H 6700 2150 50  0001 C CNN
 	1    6700 2150
@@
 F 0 "R68" V 6205 1900 50  0000 C CNN
 F 1 "100k" V 6114 1900 50  0000 C CNN
-F 2 "Resistor_SMD:R_0603_1608Metric_Pad1.05x0.95mm_HandSolder" V 6040 1890 50  0001 C CNN
+F 2 "Resistor_SMD:R_0805_2012Metric" V 6040 1890 50  0001 C CNN
 F 3 "~" H 6000 1900 50  0001 C CNN
 	1    6000 1900
@@
 F 0 "R63" H 5818 2296 50  0000 L CNN
 F 1 "10k" H 5818 2205 50  0000 L CNN
-F 2 "Resistor_SMD:R_0603_1608Metric_Pad1.05x0.95mm_HandSolder" V 5790 2240 50  0001 C CNN
+F 2 "Resistor_SMD:R_0805_2012Metric" V 5790 2240 50  0001 C CNN
 F 3 "~" H 5750 2250 50  0001 C CNN
 	1    5750 2250
@@
 F 0 "R72" H 6632 3604 50  0000 R CNN
 F 1 "100k" H 6632 3695 50  0000 R CNN
-F 2 "Resistor_SMD:R_0603_1608Metric_Pad1.05x0.95mm_HandSolder" V 6740 3640 50  0001 C CNN
+F 2 "Resistor_SMD:R_0805_2012Metric" V 6740 3640 50  0001 C CNN
 F 3 "~" H 6700 3650 50  0001 C CNN
 	1    6700 3650
@@
 F 0 "R76" V 6205 3400 50  0000 C CNN
 F 1 "100k" V 6114 3400 50  0000 C CNN
-F 2 "Resistor_SMD:R_0603_1608Metric_Pad1.05x0.95mm_HandSolder" V 6040 3390 50  0001 C CNN
+F 2 "Resistor_SMD:R_0805_2012Metric" V 6040 3390 50  0001 C CNN
 F 3 "~" H 6000 3400 50  0001 C CNN
 	1    6000 3400
@@
 F 0 "R61" H 5818 3796 50  0000 L CNN
 F 1 "10k" H 5818 3705 50  0000 L CNN
-F 2 "Resistor_SMD:R_0603_1608Metric_Pad1.05x0.95mm_HandSolder" V 5790 3740 50  0001 C CNN
+F 2 "Resistor_SMD:R_0805_2012Metric" V 5790 3740 50  0001 C CNN
 F 3 "~" H 5750 3750 50  0001 C CNN
 	1    5750 3750
@@
 F 0 "R70" H 10132 2104 50  0000 R CNN
 F 1 "100k" H 10132 2195 50  0000 R CNN
-F 2 "Resistor_SMD:R_0603_1608Metric_Pad1.05x0.95mm_HandSolder" V 10240 2140 50  0001 C CNN
+F 2 "Resistor_SMD:R_0805_2012Metric" V 10240 2140 50  0001 C CNN
 F 3 "~" H 10200 2150 50  0001 C CNN
 	1    10200 2150
@@
 F 0 "R67" V 9705 1900 50  0000 C CNN
 F 1 "100k" V 9614 1900 50  0000 C CNN
-F 2 "Resistor_SMD:R_0603_1608Metric_Pad1.05x0.95mm_HandSolder" V 9540 1890 50  0001 C CNN
+F 2 "Resistor_SMD:R_0805_2012Metric" V 9540 1890 50  0001 C CNN
 F 3 "~" H 9500 1900 50  0001 C CNN
 	1    9500 1900
@@
 F 0 "R64" H 9318 2296 50  0000 L CNN
 F 1 "10k" H 9318 2205 50  0000 L CNN
-F 2 "Resistor_SMD:R_0603_1608Metric_Pad1.05x0.95mm_HandSolder" V 9290 2240 50  0001 C CNN
+F 2 "Resistor_SMD:R_0805_2012Metric" V 9290 2240 50  0001 C CNN
 F 3 "~" H 9250 2250 50  0001 C CNN
 	1    9250 2250
@@
 F 0 "R74" H 10132 3604 50  0000 R CNN
 F 1 "100k" H 10132 3695 50  0000 R CNN
-F 2 "Resistor_SMD:R_0603_1608Metric_Pad1.05x0.95mm_HandSolder" V 10240 3640 50  0001 C CNN
+F 2 "Resistor_SMD:R_0805_2012Metric" V 10240 3640 50  0001 C CNN
 F 3 "~" H 10200 3650 50  0001 C CNN
 	1    10200 3650
@@
 F 0 "R75" V 9705 3400 50  0000 C CNN
 F 1 "100k" V 9614 3400 50  0000 C CNN
-F 2 "Resistor_SMD:R_0603_1608Metric_Pad1.05x0.95mm_HandSolder" V 9540 3390 50  0001 C CNN
+F 2 "Resistor_SMD:R_0805_2012Metric" V 9540 3390 50  0001 C CNN
 F 3 "~" H 9500 3400 50  0001 C CNN
 	1    9500 3400
@@
 F 0 "R60" H 9318 3796 50  0000 L CNN
 F 1 "10k" H 9318 3705 50  0000 L CNN
-F 2 "Resistor_SMD:R_0603_1608Metric_Pad1.05x0.95mm_HandSolder" V 9290 3740 50  0001 C CNN
+F 2 "Resistor_SMD:R_0805_2012Metric" V 9290 3740 50  0001 C CNN
 F 3 "~" H 9250 3750 50  0001 C CNN
 	1    9250 3750
