File: DAC&CV Outputs.sch (KiCad schematic (older format))
At the start: 57 parts, among them IC12 TL074, IC13 TL074, IC14 TL074, IC4 DAC8168, J1 -8.1V to 8.1V, J2 -8.1V to 8.1V, J3 -8.1V to 8.1V, J4 -8.1V to 8.1V, J5 -8.1V to 8.1V, J6 -8.1V to 8.1V

Commit message: Progress on routing tracks
Most of the power tracks are routed
Parts:
- C18, C43, C44, C45, C46, C47, C48, C49, C50, C51, C52, C53, C54, C55: footprint Capacitor_SMD:C_0603_1608Metric_Pad1.05x0.95mm_HandSolder -> Capacitor_SMD:C_0805_2012Metric
- C22: footprint Capacitor_SMD:C_1206_3216Metric_Pad1.42x1.75mm_HandSolder -> Capacitor_SMD:C_1206_3216Metric
- R34, R35, R36, R37, R38, R39, R40, R41, R42, R43, R44, R45, R46, R47, R48, R49, R50, R51, R52, R53, R54, R55, R56, R57, R58, R59: footprint Resistor_SMD:R_0603_1608Metric_Pad1.05x0.95mm_HandSolder -> Resistor_SMD:R_0805_2012Metric

Commit message: Re-orientation
Fixed some bad op-amp orientations
Changed lines of the file:
@@
 U 4 1 5BFBE4FC
 P 1800 1800
-F 0 "IC14" H 1800 2167 50  0000 C CNN
-F 1 "TL074" H 1800 2076 50  0000 C CNN
+F 0 "IC14" H 1800 1433 50  0000 C CNN
+F 1 "TL074" H 1800 1524 50  0000 C CNN
 F 2 "Package_SO:TSSOP-14_4.4x5mm_P0.65mm" H 1750 1900 50  0001 C CNN
 F 3 "http://www.ti.com/lit/ds/symlink/tl071.pdf" H 1850 2000 50  0001 C CNN
 	4    1800 1800
-	1    0    0    -1
+	1    0    0    1
 $EndComp
 $Comp
@@
 U 3 1 5BFBE55B
 P 1900 2900
-F 0 "IC14" H 1900 3267 50  0000 C CNN
-F 1 "TL074" H 1900 3176 50  0000 C CNN
+F 0 "IC14" H 1900 3150 50  0000 C CNN
+F 1 "TL074" H 1900 3250 50  0000 C CNN
 F 2 "Package_SO:TSSOP-14_4.4x5mm_P0.65mm" H 1850 3000 50  0001 C CNN
 F 3 "http://www.ti.com/lit/ds/symlink/tl071.pdf" H 1950 3100 50  0001 C CNN
 	3    1900 2900
-	1    0    0    -1
+	1    0    0    1
 $EndComp
 $Comp
@@
 U 4 1 5BFC7399
 P 4900 1800
-F 0 "IC13" H 4900 2167 50  0000 C CNN
-F 1 "TL074" H 4900 2076 50  0000 C CNN
+F 0 "IC13" H 4900 1433 50  0000 C CNN
+F 1 "TL074" H 4900 1524 50  0000 C CNN
 F 2 "Package_SO:TSSOP-14_4.4x5mm_P0.65mm" H 4850 1900 50  0001 C CNN
 F 3 "http://www.ti.com/lit/ds/symlink/tl071.pdf" H 4950 2000 50  0001 C CNN
 	4    4900 1800
-	1    0    0    -1
+	1    0    0    1
 $EndComp
 $Comp
@@
 U 3 1 5BFC73A0
 P 5000 2900
-F 0 "IC13" H 5000 3267 50  0000 C CNN
-F 1 "TL074" H 5000 3176 50  0000 C CNN
+F 0 "IC13" H 5000 3150 50  0000 C CNN
+F 1 "TL074" H 5000 3250 50  0000 C CNN
 F 2 "Package_SO:TSSOP-14_4.4x5mm_P0.65mm" H 4950 3000 50  0001 C CNN
 F 3 "http://www.ti.com/lit/ds/symlink/tl071.pdf" H 5050 3100 50  0001 C CNN
 	3    5000 2900
-	1    0    0    -1
+	1    0    0    1
 $EndComp
 $Comp
@@
 U 4 1 5BFCBAA5
 P 8000 1800
-F 0 "IC12" H 8000 2167 50  0000 C CNN
-F 1 "TL074" H 8000 2076 50  0000 C CNN
+F 0 "IC12" H 8000 1433 50  0000 C CNN
+F 1 "TL074" H 8000 1524 50  0000 C CNN
 F 2 "Package_SO:TSSOP-14_4.4x5mm_P0.65mm" H 7950 1900 50  0001 C CNN
 F 3 "http://www.ti.com/lit/ds/symlink/tl071.pdf" H 8050 2000 50  0001 C CNN
 	4    8000 1800
-	1    0    0    -1
+	1    0    0    1
 $EndComp
 $Comp
@@
 U 3 1 5BFCBAAC
 P 8100 2900
-F 0 "IC12" H 8100 3267 50  0000 C CNN
-F 1 "TL074" H 8100 3176 50  0000 C CNN
+F 0 "IC12" H 8100 3150 50  0000 C CNN
+F 1 "TL074" H 8100 3250 50  0000 C CNN
 F 2 "Package_SO:TSSOP-14_4.4x5mm_P0.65mm" H 8050 3000 50  0001 C CNN
 F 3 "http://www.ti.com/lit/ds/symlink/tl071.pdf" H 8150 3100 50  0001 C CNN
 	3    8100 2900
-	1    0    0    -1
-$EndComp
-$Comp
+	1    0    0    1
+$EndComp
+$Comp
