File: CV Inputs.sch (KiCad schematic (older format))
At the start: 42 parts, among them IC10 MCP6002, IC8 MCP6002, IC9 MCP6002, J13 -81V to 8.1V, J14 -81V to 8.1V, J15 -81V to 8.1V, J16 -81V to 8.1V, J17 -81V to 8.1V, J18 -81V to 8.1V

Commit message: Rough Placement Completed
Completed the rough placement of the components on the pcb
Parts:
- IC10, IC8, IC9: footprint Package_SO:MSOP-8-1EP_3x3mm_P0.65mm_EP2.54x2.8mm -> Package_SO:SOIC-8_3.9x4.9mm_P1.27mm
Changed lines of the file:
@@
 F 0 "IC10" H 3100 4583 50  0000 C CNN
 F 1 "MCP6002" H 3100 4674 50  0000 C CNN
-F 2 "Package_SO:MSOP-8-1EP_3x3mm_P0.65mm_EP2.54x2.8mm" H 3100 4950 50  0001 C CNN
+F 2 "Package_SO:SOIC-8_3.9x4.9mm_P1.27mm" H 3100 4950 50  0001 C CNN
 F 3 "http://ww1.microchip.com/downloads/en/DeviceDoc/21733j.pdf" H 3100 4950 50  0001 C CNN
 	1    3100 4950
@@
 F 0 "IC10" H 3100 2883 50  0000 C CNN
 F 1 "MCP6002" H 3100 2974 50  0000 C CNN
-F 2 "Package_SO:MSOP-8-1EP_3x3mm_P0.65mm_EP2.54x2.8mm" H 3100 3250 50  0001 C CNN
+F 2 "Package_SO:SOIC-8_3.9x4.9mm_P1.27mm" H 3100 3250 50  0001 C CNN
 F 3 "http://ww1.microchip.com/downloads/en/DeviceDoc/21733j.pdf" H 3100 3250 50  0001 C CNN
 	2    3100 3250
@@
 F 0 "IC9" H 6050 4583 50  0000 C CNN
 F 1 "MCP6002" H 6050 4674 50  0000 C CNN
-F 2 "Package_SO:MSOP-8-1EP_3x3mm_P0.65mm_EP2.54x2.8mm" H 6050 4950 50  0001 C CNN
+F 2 "Package_SO:SOIC-8_3.9x4.9mm_P1.27mm" H 6050 4950 50  0001 C CNN
 F 3 "http://ww1.microchip.com/downloads/en/DeviceDoc/21733j.pdf" H 6050 4950 50  0001 C CNN
 	1    6050 4950
@@
 F 0 "IC9" H 6050 2883 50  0000 C CNN
 F 1 "MCP6002" H 6050 2974 50  0000 C CNN
-F 2 "Package_SO:MSOP-8-1EP_3x3mm_P0.65mm_EP2.54x2.8mm" H 6050 3250 50  0001 C CNN
+F 2 "Package_SO:SOIC-8_3.9x4.9mm_P1.27mm" H 6050 3250 50  0001 C CNN
 F 3 "http://ww1.microchip.com/downloads/en/DeviceDoc/21733j.pdf" H 6050 3250 50  0001 C CNN
 	2    6050 3250
@@
 F 0 "IC8" H 9000 4583 50  0000 C CNN
 F 1 "MCP6002" H 9000 4674 50  0000 C CNN
-F 2 "Package_SO:MSOP-8-1EP_3x3mm_P0.65mm_EP2.54x2.8mm" H 9000 4950 50  0001 C CNN
+F 2 "Package_SO:SOIC-8_3.9x4.9mm_P1.27mm" H 9000 4950 50  0001 C CNN
 F 3 "http://ww1.microchip.com/downloads/en/DeviceDoc/21733j.pdf" H 9000 4950 50  0001 C CNN
 	1    9000 4950
@@
 F 0 "IC8" H 9000 2883 50  0000 C CNN
 F 1 "MCP6002" H 9000 2974 50  0000 C CNN
-F 2 "Package_SO:MSOP-8-1EP_3x3mm_P0.65mm_EP2.54x2.8mm" H 9000 3250 50  0001 C CNN
+F 2 "Package_SO:SOIC-8_3.9x4.9mm_P1.27mm" H 9000 3250 50  0001 C CNN
 F 3 "http://ww1.microchip.com/downloads/en/DeviceDoc/21733j.pdf" H 9000 3250 50  0001 C CNN
 	2    9000 3250
@@
 F 0 "IC10" H 2358 6546 50  0000 L CNN
 F 1 "MCP6002" H 2358 6455 50  0000 L CNN
-F 2 "Package_SO:MSOP-8-1EP_3x3mm_P0.65mm_EP2.54x2.8mm" H 2400 6500 50  0001 C CNN
+F 2 "Package_SO:SOIC-8_3.9x4.9mm_P1.27mm" H 2400 6500 50  0001 C CNN
 F 3 "http://ww1.microchip.com/downloads/en/DeviceDoc/21733j.pdf" H 2400 6500 50  0001 C CNN
 	3    2400 6500
@@
 F 0 "IC9" H 2858 6546 50  0000 L CNN
 F 1 "MCP6002" H 2858 6455 50  0000 L CNN
-F 2 "Package_SO:MSOP-8-1EP_3x3mm_P0.65mm_EP2.54x2.8mm" H 2900 6500 50  0001 C CNN
+F 2 "Package_SO:SOIC-8_3.9x4.9mm_P1.27mm" H 2900 6500 50  0001 C CNN
 F 3 "http://ww1.microchip.com/downloads/en/DeviceDoc/21733j.pdf" H 2900 6500 50  0001 C CNN
 	3    2900 6500
@@
 F 0 "IC8" H 3358 6546 50  0000 L CNN
 F 1 "MCP6002" H 3358 6455 50  0000 L CNN
-F 2 "Package_SO:MSOP-8-1EP_3x3mm_P0.65mm_EP2.54x2.8mm" H 3400 6500 50  0001 C CNN
+F 2 "Package_SO:SOIC-8_3.9x4.9mm_P1.27mm" H 3400 6500 50  0001 C CNN
 F 3 "http://ww1.microchip.com/downloads/en/DeviceDoc/21733j.pdf" H 3400 6500 50  0001 C CNN
 	3    3400 6500

Commit message: Progress on routing tracks
Most of the power tracks are routed
Parts:
- C27, C28, C29, C30, C31, C32, C33, C34, C35, C36, C37, C38, C39, C40, C42: footprint Capacitor_SMD:C_0603_1608Metric_Pad1.05x0.95mm_HandSolder -> Capacitor_SMD:C_0805_2012Metric
- R13, R14, R15, R16, R19, R20, R21, R22, R23, R24, R25, R26, R27, R28, R29, R30, R31, R32: footprint Resistor_SMD:R_0603_1608Metric_Pad1.05x0.95mm_HandSolder -> Resistor_SMD:R_0805_2012Metric
Changed lines of the file:
@@
 F 0 "R14" V 2895 4450 50  0000 C CNN
 F 1 "20k" V 2986 4450 50  0000 C CNN
-F 2 "Resistor_SMD:R_0603_1608Metric_Pad1.05x0.95mm_HandSolder" V 3140 4440 50  0001 C CNN
+F 2 "Resistor_SMD:R_0805_2012Metric" V 3140 4440 50  0001 C CNN
 F 3 "~" H 3100 4450 50  0001 C CNN
 	1    3100 4450
@@
 F 0 "R21" V 2345 4400 50  0000 C CNN
 F 1 "30k" V 2436 4400 50  0000 C CNN
-F 2 "Resistor_SMD:R_0603_1608Metric_Pad1.05x0.95mm_HandSolder" V 2590 4390 50  0001 C CNN
+F 2 "Resistor_SMD:R_0805_2012Metric" V 2590 4390 50  0001 C CNN
 F 3 "~" H 2550 4400 50  0001 C CNN
 	1    2550 4400
@@
 F 0 "R28" V 2345 4850 50  0000 C CNN
 F 1 "100k" V 2436 4850 50  0000 C CNN
-F 2 "Resistor_SMD:R_0603_1608Metric_Pad1.05x0.95mm_HandSolder" V 2590 4840 50  0001 C CNN
+F 2 "Resistor_SMD:R_0805_2012Metric" V 2590 4840 50  0001 C CNN
 F 3 "~" H 2550 4850 50  0001 C CNN
 	1    2550 4850
@@
 F 0 "C32" V 2848 4100 50  0000 C CNN
 F 1 "2.2n" V 2939 4100 50  0000 C CNN
-F 2 "Capacitor_SMD:C_0603_1608Metric_Pad1.05x0.95mm_HandSolder" H 3100 4100 50  0001 C CNN
+F 2 "Capacitor_SMD:C_0805_2012Metric" H 3100 4100 50  0001 C CNN
 F 3 "~" H 3100 4100 50  0001 C CNN
 	1    3100 4100
@@
 F 0 "C39" H 2465 5096 50  0000 L CNN
 F 1 "ESD" H 2465 5005 50  0000 L CNN
-F 2 "Capacitor_SMD:C_0603_1608Metric_Pad1.05x0.95mm_HandSolder" H 2350 5050 50  0001 C CNN
+F 2 "Capacitor_SMD:C_0805_2012Metric" H 2350 5050 50  0001 C CNN
 F 3 "~" H 2350 5050 50  0001 C CNN
 	1    2350 5050
@@
 F 0 "R16" V 2895 2750 50  0000 C CNN
 F 1 "20k" V 2986 2750 50  0000 C CNN
-F 2 "Resistor_SMD:R_0603_1608Metric_Pad1.05x0.95mm_HandSolder" V 3140 2740 50  0001 C CNN
+F 2 "Resistor_SMD:R_0805_2012Metric" V 3140 2740 50  0001 C CNN
 F 3 "~" H 3100 2750 50  0001 C CNN
 	1    3100 2750
@@
 F 0 "R29" V 2345 2700 50  0000 C CNN
 F 1 "30k" V 2436 2700 50  0000 C CNN
-F 2 "Resistor_SMD:R_0603_1608Metric_Pad1.05x0.95mm_HandSolder" V 2590 2690 50  0001 C CNN
+F 2 "Resistor_SMD:R_0805_2012Metric" V 2590 2690 50  0001 C CNN
 F 3 "~" H 2550 2700 50  0001 C CNN
 	1    2550 2700
@@
 F 0 "R30" V 2345 3150 50  0000 C CNN
 F 1 "100k" V 2436 3150 50  0000 C CNN
-F 2 "Resistor_SMD:R_0603_1608Metric_Pad1.05x0.95mm_HandSolder" V 2590 3140 50  0001 C CNN
+F 2 "Resistor_SMD:R_0805_2012Metric" V 2590 3140 50  0001 C CNN
 F 3 "~" H 2550 3150 50  0001 C CNN
 	1    2550 3150
@@
 F 0 "C35" V 2848 2400 50  0000 C CNN
 F 1 "2.2n" V 2939 2400 50  0000 C CNN
-F 2 "Capacitor_SMD:C_0603_1608Metric_Pad1.05x0.95mm_HandSolder" H 3100 2400 50  0001 C CNN
+F 2 "Capacitor_SMD:C_0805_2012Metric" H 3100 2400 50  0001 C CNN
 F 3 "~" H 3100 2400 50  0001 C CNN
 	1    3100 2400
@@
 F 0 "C38" H 2465 3396 50  0000 L CNN
 F 1 "ESD" H 2465 3305 50  0000 L CNN
-F 2 "Capacitor_SMD:C_0603_1608Metric_Pad1.05x0.95mm_HandSolder" H 2350 3350 50  0001 C CNN
+F 2 "Capacitor_SMD:C_0805_2012Metric" H 2350 3350 50  0001 C CNN
 F 3 "~" H 2350 3350 50  0001 C CNN
 	1    2350 3350
@@
 F 0 "R15" V 5845 4450 50  0000 C CNN
 F 1 "20k" V 5936 4450 50  0000 C CNN
-F 2 "Resistor_SMD:R_0603_1608Metric_Pad1.05x0.95mm_HandSolder" V 6090 4440 50  0001 C CNN
+F 2 "Resistor_SMD:R_0805_2012Metric" V 6090 4440 50  0001 C CNN
 F 3 "~" H 6050 4450 50  0001 C CNN
 	1    6050 4450
@@
 F 0 "R22" V 5295 4400 50  0000 C CNN
 F 1 "30k" V 5386 4400 50  0000 C CNN
-F 2 "Resistor_SMD:R_0603_1608Metric_Pad1.05x0.95mm_HandSolder" V 5540 4390 50  0001 C CNN
+F 2 "Resistor_SMD:R_0805_2012Metric" V 5540 4390 50  0001 C CNN
 F 3 "~" H 5500 4400 50  0001 C CNN
 	1    5500 4400
@@
 F 0 "R25" V 5295 4850 50  0000 C CNN
 F 1 "100k" V 5386 4850 50  0000 C CNN
-F 2 "Resistor_SMD:R_0603_1608Metric_Pad1.05x0.95mm_HandSolder" V 5540 4840 50  0001 C CNN
+F 2 "Resistor_SMD:R_0805_2012Metric" V 5540 4840 50  0001 C CNN
 F 3 "~" H 5500 4850 50  0001 C CNN
 	1    5500 4850
@@
 F 0 "C29" V 5798 4100 50  0000 C CNN
 F 1 "2.2n" V 5889 4100 50  0000 C CNN
-F 2 "Capacitor_SMD:C_0603_1608Metric_Pad1.05x0.95mm_HandSolder" H 6050 4100 50  0001 C CNN
+F 2 "Capacitor_SMD:C_0805_2012Metric" H 6050 4100 50  0001 C CNN
 F 3 "~" H 6050 4100 50  0001 C CNN
 	1    6050 4100
@@
 F 0 "C40" H 5415 5096 50  0000 L CNN
 F 1 "ESD" H 5415 5005 50  0000 L CNN
-F 2 "Capacitor_SMD:C_0603_1608Metric_Pad1.05x0.95mm_HandSolder" H 5300 5050 50  0001 C CNN
+F 2 "Capacitor_SMD:C_0805_2012Metric" H 5300 5050 50  0001 C CNN
 F 3 "~" H 5300 5050 50  0001 C CNN
 	1    5300 5050
@@
 F 0 "R13" V 5845 2750 50  0000 C CNN
 F 1 "20k" V 5936 2750 50  0000 C CNN
-F 2 "Resistor_SMD:R_0603_1608Metric_Pad1.05x0.95mm_HandSolder" V 6090 2740 50  0001 C CNN
+F 2 "Resistor_SMD:R_0805_2012Metric" V 6090 2740 50  0001 C CNN
 F 3 "~" H 6050 2750 50  0001 C CNN
 	1    6050 2750
@@
 F 0 "R26" V 5295 2700 50  0000 C CNN
 F 1 "30k" V 5386 2700 50  0000 C CNN
-F 2 "Resistor_SMD:R_0603_1608Metric_Pad1.05x0.95mm_HandSolder" V 5540 2690 50  0001 C CNN
+F 2 "Resistor_SMD:R_0805_2012Metric" V 5540 2690 50  0001 C CNN
 F 3 "~" H 5500 2700 50  0001 C CNN
 	1    5500 2700
@@
 F 0 "R27" V 5295 3150 50  0000 C CNN
 F 1 "100k" V 5386 3150 50  0000 C CNN
-F 2 "Resistor_SMD:R_0603_1608Metric_Pad1.05x0.95mm_HandSolder" V 5540 3140 50  0001 C CNN
+F 2 "Resistor_SMD:R_0805_2012Metric" V 5540 3140 50  0001 C CNN
 F 3 "~" H 5500 3150 50  0001 C CNN
 	1    5500 3150
@@
 F 0 "C31" V 5798 2400 50  0000 C CNN
 F 1 "2.2n" V 5889 2400 50  0000 C CNN
-F 2 "Capacitor_SMD:C_0603_1608Metric_Pad1.05x0.95mm_HandSolder" H 6050 2400 50  0001 C CNN
+F 2 "Capacitor_SMD:C_0805_2012Metric" H 6050 2400 50  0001 C CNN
 F 3 "~" H 6050 2400 50  0001 C CNN
 	1    6050 2400
@@
 F 0 "C37" H 5415 3396 50  0000 L CNN
 F 1 "ESD" H 5415 3305 50  0000 L CNN
-F 2 "Capacitor_SMD:C_0603_1608Metric_Pad1.05x0.95mm_HandSolder" H 5300 3350 50  0001 C CNN
+F 2 "Capacitor_SMD:C_0805_2012Metric" H 5300 3350 50  0001 C CNN
 F 3 "~" H 5300 3350 50  0001 C CNN
 	1    5300 3350
@@
 F 0 "R20" V 8795 4450 50  0000 C CNN
 F 1 "20k" V 8886 4450 50  0000 C CNN
-F 2 "Resistor_SMD:R_0603_1608Metric_Pad1.05x0.95mm_HandSolder" V 9040 4440 50  0001 C CNN
+F 2 "Resistor_SMD:R_0805_2012Metric" V 9040 4440 50  0001 C CNN
 F 3 "~" H 9000 4450 50  0001 C CNN
 	1    9000 4450
@@
 F 0 "R23" V 8245 4400 50  0000 C CNN
 F 1 "30k" V 8336 4400 50  0000 C CNN
-F 2 "Resistor_SMD:R_0603_1608Metric_Pad1.05x0.95mm_HandSolder" V 8490 4390 50  0001 C CNN
+F 2 "Resistor_SMD:R_0805_2012Metric" V 8490 4390 50  0001 C CNN
 F 3 "~" H 8450 4400 50  0001 C CNN
 	1    8450 4400
@@
 F 0 "R32" V 8245 4850 50  0000 C CNN
 F 1 "100k" V 8336 4850 50  0000 C CNN
-F 2 "Resistor_SMD:R_0603_1608Metric_Pad1.05x0.95mm_HandSolder" V 8490 4840 50  0001 C CNN
+F 2 "Resistor_SMD:R_0805_2012Metric" V 8490 4840 50  0001 C CNN
 F 3 "~" H 8450 4850 50  0001 C CNN
 	1    8450 4850
@@
 F 0 "C28" V 8748 4100 50  0000 C CNN
 F 1 "470p" V 8839 4100 50  0000 C CNN
-F 2 "Capacitor_SMD:C_0603_1608Metric_Pad1.05x0.95mm_HandSolder" H 9000 4100 50  0001 C CNN
+F 2 "Capacitor_SMD:C_0805_2012Metric" H 9000 4100 50  0001 C CNN
 F 3 "~" H 9000 4100 50  0001 C CNN
 	1    9000 4100
@@
 F 0 "C42" H 8365 5096 50  0000 L CNN
 F 1 "ESD" H 8365 5005 50  0000 L CNN
-F 2 "Capacitor_SMD:C_0603_1608Metric_Pad1.05x0.95mm_HandSolder" H 8250 5050 50  0001 C CNN
+F 2 "Capacitor_SMD:C_0805_2012Metric" H 8250 5050 50  0001 C CNN
 F 3 "~" H 8250 5050 50  0001 C CNN
 	1    8250 5050
@@
 F 0 "R19" V 8795 2750 50  0000 C CNN
 F 1 "20k" V 8886 2750 50  0000 C CNN
-F 2 "Resistor_SMD:R_0603_1608Metric_Pad1.05x0.95mm_HandSolder" V 9040 2740 50  0001 C CNN
+F 2 "Resistor_SMD:R_0805_2012Metric" V 9040 2740 50  0001 C CNN
 F 3 "~" H 9000 2750 50  0001 C CNN
 	1    9000 2750
@@
 F 0 "R24" V 8245 2700 50  0000 C CNN
 F 1 "30k" V 8336 2700 50  0000 C CNN
-F 2 "Resistor_SMD:R_0603_1608Metric_Pad1.05x0.95mm_HandSolder" V 8490 2690 50  0001 C CNN
+F 2 "Resistor_SMD:R_0805_2012Metric" V 8490 2690 50  0001 C CNN
 F 3 "~" H 8450 2700 50  0001 C CNN
 	1    8450 2700
@@
 F 0 "R31" V 8245 3150 50  0000 C CNN
 F 1 "100k" V 8336 3150 50  0000 C CNN
-F 2 "Resistor_SMD:R_0603_1608Metric_Pad1.05x0.95mm_HandSolder" V 8490 3140 50  0001 C CNN
+F 2 "Resistor_SMD:R_0805_2012Metric" V 8490 3140 50  0001 C CNN
 F 3 "~" H 8450 3150 50  0001 C CNN
 	1    8450 3150
@@
 F 0 "C27" V 8748 2400 50  0000 C CNN
 F 1 "2.2n" V 8839 2400 50  0000 C CNN
-F 2 "Capacitor_SMD:C_0603_1608Metric_Pad1.05x0.95mm_HandSolder" H 9000 2400 50  0001 C CNN
+F 2 "Capacitor_SMD:C_0805_2012Metric" H 9000 2400 50  0001 C CNN
 F 3 "~" H 9000 2400 50  0001 C CNN
 	1    9000 2400
@@
 F 0 "C36" H 8365 3396 50  0000 L CNN
 F 1 "ESD" H 8365 3305 50  0000 L CNN
-F 2 "Capacitor_SMD:C_0603_1608Metric_Pad1.05x0.95mm_HandSolder" H 8250 3350 50  0001 C CNN
+F 2 "Capacitor_SMD:C_0805_2012Metric" H 8250 3350 50  0001 C CNN
 F 3 "~" H 8250 3350 50  0001 C CNN
 	1    8250 3350
@@
 F 0 "C33" H 4015 6546 50  0000 L CNN
 F 1 "100n" H 4015 6455 50  0000 L CNN
-F 2 "Capacitor_SMD:C_0603_1608Metric_Pad1.05x0.95mm_HandSolder" H 3900 6500 50  0001 C CNN
+F 2 "Capacitor_SMD:C_0805_2012Metric" H 3900 6500 50  0001 C CNN
 F 3 "~" H 3900 6500 50  0001 C CNN
 	1    3900 6500
@@
 F 0 "C30" H 4415 6546 50  0000 L CNN
 F 1 "100n" H 4415 6455 50  0000 L CNN
-F 2 "Capacitor_SMD:C_0603_1608Metric_Pad1.05x0.95mm_HandSolder" H 4300 6500 50  0001 C CNN
+F 2 "Capacitor_SMD:C_0805_2012Metric" H 4300 6500 50  0001 C CNN
 F 3 "~" H 4300 6500 50  0001 C CNN
 	1    4300 6500
@@
 F 0 "C34" H 4815 6546 50  0000 L CNN
 F 1 "100n" H 4815 6455 50  0000 L CNN
-F 2 "Capacitor_SMD:C_0603_1608Metric_Pad1.05x0.95mm_HandSolder" H 4700 6500 50  0001 C CNN
+F 2 "Capacitor_SMD:C_0805_2012Metric" H 4700 6500 50  0001 C CNN
 F 3 "~" H 4700 6500 50  0001 C CNN
 	1    4700 6500

Commit message: Added Mounting Holes
Parts:
- J13, J14, J15, J16, J17, J18: value -81V to 8.1V -> -8.1V to 8.1V
Changed lines of the file:
@@
 P 1850 4950
 F 0 "J14" H 1854 5228 50  0000 C CNN
-F 1 "-81V to 8.1V" H 1854 5137 50  0000 C CNN
+F 1 "-8.1V to 8.1V" H 1854 5137 50  0000 C CNN
 F 2 "WQP-PJ301M-12_JACK:WQP-PJ301M-12_JACK" H 1850 4950 50  0001 L BNN
 F 3 "" H 1850 4950 50  0001 C CNN
@@
 P 1850 3250
 F 0 "J13" H 1854 3528 50  0000 C CNN
-F 1 "-81V to 8.1V" H 1854 3437 50  0000 C CNN
+F 1 "-8.1V to 8.1V" H 1854 3437 50  0000 C CNN
 F 2 "WQP-PJ301M-12_JACK:WQP-PJ301M-12_JACK" H 1850 3250 50  0001 L BNN
 F 3 "" H 1850 3250 50  0001 C CNN
@@
 P 4800 4950
 F 0 "J16" H 4804 5228 50  0000 C CNN
-F 1 "-81V to 8.1V" H 4804 5137 50  0000 C CNN
+F 1 "-8.1V to 8.1V" H 4804 5137 50  0000 C CNN
 F 2 "WQP-PJ301M-12_JACK:WQP-PJ301M-12_JACK" H 4800 4950 50  0001 L BNN
 F 3 "" H 4800 4950 50  0001 C CNN
@@
 P 4800 3250
 F 0 "J15" H 4804 3528 50  0000 C CNN
-F 1 "-81V to 8.1V" H 4804 3437 50  0000 C CNN
+F 1 "-8.1V to 8.1V" H 4804 3437 50  0000 C CNN
 F 2 "WQP-PJ301M-12_JACK:WQP-PJ301M-12_JACK" H 4800 3250 50  0001 L BNN
 F 3 "" H 4800 3250 50  0001 C CNN
@@
 P 7750 4950
 F 0 "J18" H 7754 5228 50  0000 C CNN
-F 1 "-81V to 8.1V" H 7754 5137 50  0000 C CNN
+F 1 "-8.1V to 8.1V" H 7754 5137 50  0000 C CNN
 F 2 "WQP-PJ301M-12_JACK:WQP-PJ301M-12_JACK" H 7750 4950 50  0001 L BNN
 F 3 "" H 7750 4950 50  0001 C CNN
@@
 P 7750 3250
 F 0 "J17" H 7754 3528 50  0000 C CNN
-F 1 "-81V to 8.1V" H 7754 3437 50  0000 C CNN
+F 1 "-8.1V to 8.1V" H 7754 3437 50  0000 C CNN
 F 2 "WQP-PJ301M-12_JACK:WQP-PJ301M-12_JACK" H 7750 3250 50  0001 L BNN
 F 3 "" H 7750 3250 50  0001 C CNN
