File: MCU.sch (KiCad schematic (older format))
At the start: 21 parts, among them IC5 STM32F373RBTx, Q1 8MHz

Commit message: Progress on routing tracks
Most of the power tracks are routed
Parts:
- C11, C12, C13, C14, C24, C26, C3, C4: footprint Capacitor_SMD:C_0603_1608Metric_Pad1.05x0.95mm_HandSolder -> Capacitor_SMD:C_0805_2012Metric
- C9: footprint Capacitor_SMD:C_1206_3216Metric_Pad1.42x1.75mm_HandSolder -> Capacitor_SMD:C_1206_3216Metric
- R10, R11, R12, R5, R7, R8, R9: footprint Resistor_SMD:R_0603_1608Metric_Pad1.05x0.95mm_HandSolder -> Resistor_SMD:R_0805_2012Metric
Changed lines of the file:
@@
 F 0 "C13" H 4165 1596 50  0000 L CNN
 F 1 "100n" H 4165 1505 50  0000 L CNN
-F 2 "Capacitor_SMD:C_0603_1608Metric_Pad1.05x0.95mm_HandSolder" H 4050 1550 50  0001 C CNN
+F 2 "Capacitor_SMD:C_0805_2012Metric" H 4050 1550 50  0001 C CNN
 F 3 "~" H 4050 1550 50  0001 C CNN
 	1    4050 1550
@@
 F 0 "C12" H 3765 1596 50  0000 L CNN
 F 1 "1u" H 3765 1505 50  0000 L CNN
-F 2 "Capacitor_SMD:C_0603_1608Metric_Pad1.05x0.95mm_HandSolder" H 3650 1550 50  0001 C CNN
+F 2 "Capacitor_SMD:C_0805_2012Metric" H 3650 1550 50  0001 C CNN
 F 3 "~" H 3650 1550 50  0001 C CNN
 	1    3650 1550
@@
 F 0 "C11" H 5865 1596 50  0000 L CNN
 F 1 "100n" H 5865 1505 50  0000 L CNN
-F 2 "Capacitor_SMD:C_0603_1608Metric_Pad1.05x0.95mm_HandSolder" H 5750 1550 50  0001 C CNN
+F 2 "Capacitor_SMD:C_0805_2012Metric" H 5750 1550 50  0001 C CNN
 F 3 "~" H 5750 1550 50  0001 C CNN
 	1    5750 1550
@@
 F 0 "C14" H 5465 1596 50  0000 L CNN
 F 1 "100n" H 5465 1505 50  0000 L CNN
-F 2 "Capacitor_SMD:C_0603_1608Metric_Pad1.05x0.95mm_HandSolder" H 5350 1550 50  0001 C CNN
+F 2 "Capacitor_SMD:C_0805_2012Metric" H 5350 1550 50  0001 C CNN
 F 3 "~" H 5350 1550 50  0001 C CNN
 	1    5350 1550
@@
 F 0 "C9" H 5065 1596 50  0000 L CNN
 F 1 "22u" H 5065 1505 50  0000 L CNN
-F 2 "Capacitor_SMD:C_1206_3216Metric_Pad1.42x1.75mm_HandSolder" H 4950 1550 50  0001 C CNN
+F 2 "Capacitor_SMD:C_1206_3216Metric" H 4950 1550 50  0001 C CNN
 F 3 "~" H 4950 1550 50  0001 C CNN
 	1    4950 1550
@@
 F 0 "C24" H 4165 2296 50  0000 L CNN
 F 1 "100n" H 4165 2205 50  0000 L CNN
-F 2 "Capacitor_SMD:C_0603_1608Metric_Pad1.05x0.95mm_HandSolder" H 4050 2250 50  0001 C CNN
+F 2 "Capacitor_SMD:C_0805_2012Metric" H 4050 2250 50  0001 C CNN
 F 3 "~" H 4050 2250 50  0001 C CNN
 	1    4050 2250
@@
 F 0 "C26" H 3765 2296 50  0000 L CNN
 F 1 "1u" H 3765 2205 50  0000 L CNN
-F 2 "Capacitor_SMD:C_0603_1608Metric_Pad1.05x0.95mm_HandSolder" H 3650 2250 50  0001 C CNN
+F 2 "Capacitor_SMD:C_0805_2012Metric" H 3650 2250 50  0001 C CNN
 F 3 "~" H 3650 2250 50  0001 C CNN
 	1    3650 2250
@@
 F 0 "R8" V 2705 3700 50  0000 C CNN
 F 1 "100" V 2614 3700 50  0000 C CNN
-F 2 "Resistor_SMD:R_0603_1608Metric_Pad1.05x0.95mm_HandSolder" V 2540 3690 50  0001 C CNN
+F 2 "Resistor_SMD:R_0805_2012Metric" V 2540 3690 50  0001 C CNN
 F 3 "~" H 2500 3700 50  0001 C CNN
 	1    2500 3700
@@
 F 0 "R9" V 2705 3000 50  0000 C CNN
 F 1 "100" V 2614 3000 50  0000 C CNN
-F 2 "Resistor_SMD:R_0603_1608Metric_Pad1.05x0.95mm_HandSolder" V 2540 2990 50  0001 C CNN
+F 2 "Resistor_SMD:R_0805_2012Metric" V 2540 2990 50  0001 C CNN
 F 3 "~" H 2500 3000 50  0001 C CNN
 	1    2500 3000
@@
 F 0 "C3" V 1852 3000 50  0000 C CNN
 F 1 "20p" V 1761 3000 50  0000 C CNN
-F 2 "Capacitor_SMD:C_0603_1608Metric_Pad1.05x0.95mm_HandSolder" H 1600 3000 50  0001 C CNN
+F 2 "Capacitor_SMD:C_0805_2012Metric" H 1600 3000 50  0001 C CNN
 F 3 "~" H 1600 3000 50  0001 C CNN
 	1    1600 3000
@@
 F 0 "C4" V 1852 3700 50  0000 C CNN
 F 1 "20p" V 1761 3700 50  0000 C CNN
-F 2 "Capacitor_SMD:C_0603_1608Metric_Pad1.05x0.95mm_HandSolder" H 1600 3700 50  0001 C CNN
+F 2 "Capacitor_SMD:C_0805_2012Metric" H 1600 3700 50  0001 C CNN
 F 3 "~" H 1600 3700 50  0001 C CNN
 	1    1600 3700
@@
 F 0 "R12" V 5113 2100 50  0000 C CNN
 F 1 "10k" V 5204 2100 50  0000 C CNN
-F 2 "Resistor_SMD:R_0603_1608Metric_Pad1.05x0.95mm_HandSolder" V 5040 2090 50  0001 C CNN
+F 2 "Resistor_SMD:R_0805_2012Metric" V 5040 2090 50  0001 C CNN
 F 3 "~" H 5000 2100 50  0001 C CNN
 	1    5000 2100
@@
 F 0 "R7" V 1145 5750 50  0000 C CNN
 F 1 "100" V 1236 5750 50  0000 C CNN
-F 2 "Resistor_SMD:R_0603_1608Metric_Pad1.05x0.95mm_HandSolder" V 1390 5740 50  0001 C CNN
+F 2 "Resistor_SMD:R_0805_2012Metric" V 1390 5740 50  0001 C CNN
 F 3 "~" H 1350 5750 50  0001 C CNN
 	1    1350 5750
@@
 F 0 "R5" V 1463 5850 50  0000 C CNN
 F 1 "100" V 1554 5850 50  0000 C CNN
-F 2 "Resistor_SMD:R_0603_1608Metric_Pad1.05x0.95mm_HandSolder" V 1390 5840 50  0001 C CNN
+F 2 "Resistor_SMD:R_0805_2012Metric" V 1390 5840 50  0001 C CNN
 F 3 "~" H 1350 5850 50  0001 C CNN
 	1    1350 5850
@@
 F 0 "R11" V 1145 5000 50  0000 C CNN
 F 1 "100" V 1236 5000 50  0000 C CNN
-F 2 "Resistor_SMD:R_0603_1608Metric_Pad1.05x0.95mm_HandSolder" V 1390 4990 50  0001 C CNN
+F 2 "Resistor_SMD:R_0805_2012Metric" V 1390 4990 50  0001 C CNN
 F 3 "~" H 1350 5000 50  0001 C CNN
 	1    1350 5000
@@
 F 0 "R10" V 1463 5100 50  0000 C CNN
 F 1 "100" V 1554 5100 50  0000 C CNN
-F 2 "Resistor_SMD:R_0603_1608Metric_Pad1.05x0.95mm_HandSolder" V 1390 5090 50  0001 C CNN
+F 2 "Resistor_SMD:R_0805_2012Metric" V 1390 5090 50  0001 C CNN
 F 3 "~" H 1350 5100 50  0001 C CNN
 	1    1350 5100

Commit message: Added Mounting Holes
Connections:
- wire segments 135 -> 129
Changed lines of the file:
@@
 	3650 1300 4050 1300
-Wire Wire Line
-	3250 1700 3250 1800
 Wire Wire Line
 	6350 900  6350 1900
@@
 L power:+3.3V #PWR?
 U 1 1 5BFAB98C
-P 4950 1200
+P 4750 1300
 AR Path="/5BFAB98C" Ref="#PWR?"  Part="1"
 AR Path="/5BFAB137/5BFAB98C" Ref="#PWR0106"  Part="1"
-F 0 "#PWR0106" H 4950 1050 50  0001 C CNN
-F 1 "+3.3V" H 4965 1373 50  0000 C CNN
-F 2 "" H 4950 1200 50  0001 C CNN
-F 3 "" H 4950 1200 50  0001 C CNN
-	1    4950 1200
-	1    0    0    -1
-$EndComp
-Wire Wire Line
-	4950 1200 4950 1300
+F 0 "#PWR0106" H 4750 1150 50  0001 C CNN
+F 1 "+3.3V" H 4765 1473 50  0000 C CNN
+F 2 "" H 4750 1300 50  0001 C CNN
+F 3 "" H 4750 1300 50  0001 C CNN
+	1    4750 1300
+	1    0    0    -1
+$EndComp
 Connection ~ 4950 1300
 $Comp
@@
 Connection ~ 4650 1300
 Wire Wire Line
-	3250 1800 3450 1800
-Wire Wire Line
-	3450 1800 3450 1300
-Wire Wire Line
 	3450 1300 3650 1300
 Connection ~ 3650 1300
 Wire Wire Line
-	3450 1800 3450 2000
-Wire Wire Line
 	3450 2000 3650 2000
-Connection ~ 3450 1800
 Connection ~ 3650 2000
 Wire Wire Line
@@
 $EndComp
 Wire Wire Line
-	4750 2100 4750 1300
-Wire Wire Line
 	4750 1300 4950 1300
 Text GLabel 5400 3900 0    50   Input ~ 0
@@
 Wire Wire Line
 	5400 4200 5450 4200
-Text GLabel 3250 1700 1    50   Input ~ 0
+Text GLabel 3450 1300 1    50   Input ~ 0
 +3V3_A
 Wire Wire Line
@@
 Text GLabel 1600 5100 2    50   Input ~ 0
 RIGHT_RX
+Text GLabel 1600 5850 2    50   Input ~ 0
+LEFT_TX
 Text GLabel 1600 5750 2    50   Input ~ 0
-LEFT_TX
-Text GLabel 1600 5850 2    50   Input ~ 0
 LEFT_RX
 $Comp
@@
 Wire Wire Line
 	5400 3400 5450 3400
+Text GLabel 3450 2000 1    50   Input ~ 0
++3V3_A
+$Comp
+L power:+3.3V #PWR?
+U 1 1 5C2DA1FC
+P 4750 2100
+AR Path="/5C2DA1FC" Ref="#PWR?"  Part="1"
+AR Path="/5BFAB137/5C2DA1FC" Ref="#PWR0219"  Part="1"
+F 0 "#PWR0219" H 4750 1950 50  0001 C CNN
+F 1 "+3.3V" H 4765 2273 50  0000 C CNN
+F 2 "" H 4750 2100 50  0001 C CNN
+F 3 "" H 4750 2100 50  0001 C CNN
+	1    4750 2100
+	1    0    0    -1
+$EndComp
 $EndSCHEMATC
