File: Controls.sch (KiCad schematic (older format))
At the start: 40 parts, among them IC1 TLC59281, IC3 4051, IC6 4051, SW1 SW_Push_Dual, SW2 SW_Push_Dual, SW3 SW_Push_Dual, SW4 SW_Push_Dual, SW5 SW_Push_Dual, SW6 SW_Push_Dual

Commit message: Progress on routing tracks
Most of the power tracks are routed
Parts:
- C16, C5, C7, C8: footprint Capacitor_SMD:C_0603_1608Metric_Pad1.05x0.95mm_HandSolder -> Capacitor_SMD:C_0805_2012Metric
- C6: footprint Capacitor_SMD:C_1206_3216Metric_Pad1.42x1.75mm_HandSolder -> Capacitor_SMD:C_1206_3216Metric
- L2, R1, R17, R18, R2, R3, R4, R6: footprint Resistor_SMD:R_0603_1608Metric_Pad1.05x0.95mm_HandSolder -> Resistor_SMD:R_0805_2012Metric
Changed lines of the file:
@@
 F 0 "C7" H 5815 6096 50  0000 L CNN
 F 1 "100n" H 5815 6005 50  0000 L CNN
-F 2 "Capacitor_SMD:C_0603_1608Metric_Pad1.05x0.95mm_HandSolder" H 5738 5900 50  0001 C CNN
+F 2 "Capacitor_SMD:C_0805_2012Metric" H 5738 5900 50  0001 C CNN
 F 3 "~" H 5700 6050 50  0001 C CNN
 	1    5700 6050
@@
 F 0 "C16" H 6315 6096 50  0000 L CNN
 F 1 "100n" H 6315 6005 50  0000 L CNN
-F 2 "Capacitor_SMD:C_0603_1608Metric_Pad1.05x0.95mm_HandSolder" H 6238 5900 50  0001 C CNN
+F 2 "Capacitor_SMD:C_0805_2012Metric" H 6238 5900 50  0001 C CNN
 F 3 "~" H 6200 6050 50  0001 C CNN
 	1    6200 6050
@@
 F 0 "C5" H 6815 6096 50  0000 L CNN
 F 1 "100n" H 6815 6005 50  0000 L CNN
-F 2 "Capacitor_SMD:C_0603_1608Metric_Pad1.05x0.95mm_HandSolder" H 6738 5900 50  0001 C CNN
+F 2 "Capacitor_SMD:C_0805_2012Metric" H 6738 5900 50  0001 C CNN
 F 3 "~" H 6700 6050 50  0001 C CNN
 	1    6700 6050
@@
 F 0 "R17" V 2945 950 50  0000 C CNN
 F 1 "15k" V 3036 950 50  0000 C CNN
-F 2 "Resistor_SMD:R_0603_1608Metric_Pad1.05x0.95mm_HandSolder" V 3190 940 50  0001 C CNN
+F 2 "Resistor_SMD:R_0805_2012Metric" V 3190 940 50  0001 C CNN
 F 3 "~" H 3150 950 50  0001 C CNN
 	1    3150 950
@@
 F 0 "R3" V 2945 1350 50  0000 C CNN
 F 1 "15k" V 3036 1350 50  0000 C CNN
-F 2 "Resistor_SMD:R_0603_1608Metric_Pad1.05x0.95mm_HandSolder" V 3190 1340 50  0001 C CNN
+F 2 "Resistor_SMD:R_0805_2012Metric" V 3190 1340 50  0001 C CNN
 F 3 "~" H 3150 1350 50  0001 C CNN
 	1    3150 1350
@@
 F 0 "R1" V 2945 1750 50  0000 C CNN
 F 1 "15k" V 3036 1750 50  0000 C CNN
-F 2 "Resistor_SMD:R_0603_1608Metric_Pad1.05x0.95mm_HandSolder" V 3190 1740 50  0001 C CNN
+F 2 "Resistor_SMD:R_0805_2012Metric" V 3190 1740 50  0001 C CNN
 F 3 "~" H 3150 1750 50  0001 C CNN
 	1    3150 1750
@@
 F 0 "R2" V 2945 2150 50  0000 C CNN
 F 1 "15k" V 3036 2150 50  0000 C CNN
-F 2 "Resistor_SMD:R_0603_1608Metric_Pad1.05x0.95mm_HandSolder" V 3190 2140 50  0001 C CNN
+F 2 "Resistor_SMD:R_0805_2012Metric" V 3190 2140 50  0001 C CNN
 F 3 "~" H 3150 2150 50  0001 C CNN
 	1    3150 2150
@@
 F 0 "R4" V 2945 2550 50  0000 C CNN
 F 1 "15k" V 3036 2550 50  0000 C CNN
-F 2 "Resistor_SMD:R_0603_1608Metric_Pad1.05x0.95mm_HandSolder" V 3190 2540 50  0001 C CNN
+F 2 "Resistor_SMD:R_0805_2012Metric" V 3190 2540 50  0001 C CNN
 F 3 "~" H 3150 2550 50  0001 C CNN
 	1    3150 2550
@@
 F 0 "R18" V 2945 2950 50  0000 C CNN
 F 1 "15k" V 3036 2950 50  0000 C CNN
-F 2 "Resistor_SMD:R_0603_1608Metric_Pad1.05x0.95mm_HandSolder" V 3190 2940 50  0001 C CNN
+F 2 "Resistor_SMD:R_0805_2012Metric" V 3190 2940 50  0001 C CNN
 F 3 "~" H 3150 2950 50  0001 C CNN
 	1    3150 2950
@@
 F 0 "C8" H 815 5196 50  0000 L CNN
 F 1 "100n" H 815 5105 50  0000 L CNN
-F 2 "Capacitor_SMD:C_0603_1608Metric_Pad1.05x0.95mm_HandSolder" H 738 5000 50  0001 C CNN
+F 2 "Capacitor_SMD:C_0805_2012Metric" H 738 5000 50  0001 C CNN
 F 3 "~" H 700 5150 50  0001 C CNN
 	1    700  5150
@@
 F 0 "C6" H 1215 5196 50  0000 L CNN
 F 1 "22u" H 1215 5105 50  0000 L CNN
-F 2 "Capacitor_SMD:C_1206_3216Metric_Pad1.42x1.75mm_HandSolder" H 1138 5000 50  0001 C CNN
+F 2 "Capacitor_SMD:C_1206_3216Metric" H 1138 5000 50  0001 C CNN
 F 3 "~" H 1100 5150 50  0001 C CNN
 	1    1100 5150
@@
 F 0 "L2" H 800 4746 50  0000 L CNN
 F 1 "Ferrite_Bead_Small" H 800 4655 50  0000 L CNN
-F 2 "Resistor_SMD:R_0603_1608Metric_Pad1.05x0.95mm_HandSolder" V 630 4700 50  0001 C CNN
+F 2 "Resistor_SMD:R_0805_2012Metric" V 630 4700 50  0001 C CNN
 F 3 "~" H 700 4700 50  0001 C CNN
 	1    700  4700
@@
 F 0 "R6" V 1313 5800 50  0000 C CNN
 F 1 "10k" V 1404 5800 50  0000 C CNN
-F 2 "Resistor_SMD:R_0603_1608Metric_Pad1.05x0.95mm_HandSolder" V 1240 5790 50  0001 C CNN
+F 2 "Resistor_SMD:R_0805_2012Metric" V 1240 5790 50  0001 C CNN
 F 3 "~" H 1200 5800 50  0001 C CNN
 	1    1200 5800

Commit message: Added Mounting Holes
Parts:
- removed SW1, SW2, SW3, SW4, SW5, SW6: SW_Push_Dual, Button_Switch_THT:Push E-Switch 6mm, symbol Switch:SW_Push_Dual
- added MH1, MH2, MH3: MountingHole, MountingHole:MountingHole_3.2mm_M3, symbol Mechanical:MountingHole
- added SW1, SW2, SW3, SW4, SW5, SW6: SW_Push_4pin, Button_Switch_THT:Push E-Switch 6mm, symbol Switch:SW_Push_4pin
Changed lines of the file:
@@
 Wire Wire Line
 	3400 2950 3300 2950
-$Comp
-L Switch:SW_Push_Dual SW1
-U 1 1 5C2FDCE6
-P 1300 850
-F 0 "SW1" H 1300 1135 50  0000 C CNN
-F 1 "SW_Push_Dual" H 1300 1044 50  0000 C CNN
-F 2 "Button_Switch_THT:Push E-Switch 6mm" H 1300 1050 50  0001 C CNN
-F 3 "" H 1300 1050 50  0001 C CNN
-	1    1300 850
-	1    0    0    -1
-$EndComp
 Text GLabel 1700 950  2    50   Input ~ 0
 SW_MODE_1
@@
 Wire Wire Line
 	1600 950  1600 1050
-$Comp
-L Switch:SW_Push_Dual SW2
-U 1 1 5C319EF2
-P 1300 1450
-F 0 "SW2" H 1300 1735 50  0000 C CNN
-F 1 "SW_Push_Dual" H 1300 1644 50  0000 C CNN
-F 2 "Button_Switch_THT:Push E-Switch 6mm" H 1300 1650 50  0001 C CNN
-F 3 "" H 1300 1650 50  0001 C CNN
-	1    1300 1450
-	1    0    0    -1
-$EndComp
 Text GLabel 1700 1550 2    50   Input ~ 0
 SW_MODE_2
@@
 Wire Wire Line
 	1600 1550 1600 1650
-$Comp
-L Switch:SW_Push_Dual SW3
-U 1 1 5C3220D2
-P 1300 2050
-F 0 "SW3" H 1300 2335 50  0000 C CNN
-F 1 "SW_Push_Dual" H 1300 2244 50  0000 C CNN
-F 2 "Button_Switch_THT:Push E-Switch 6mm" H 1300 2250 50  0001 C CNN
-F 3 "" H 1300 2250 50  0001 C CNN
-	1    1300 2050
-	1    0    0    -1
-$EndComp
 Text GLabel 1700 2150 2    50   Input ~ 0
 SW_MODE_3
@@
 Wire Wire Line
 	1600 2150 1600 2250
-$Comp
-L Switch:SW_Push_Dual SW4
-U 1 1 5C32B1A5
-P 1300 2650
-F 0 "SW4" H 1300 2935 50  0000 C CNN
-F 1 "SW_Push_Dual" H 1300 2844 50  0000 C CNN
-F 2 "Button_Switch_THT:Push E-Switch 6mm" H 1300 2850 50  0001 C CNN
-F 3 "" H 1300 2850 50  0001 C CNN
-	1    1300 2650
-	1    0    0    -1
-$EndComp
 Text GLabel 1700 2750 2    50   Input ~ 0
 SW_MODE_4
@@
 Wire Wire Line
 	1600 2750 1600 2850
-$Comp
-L Switch:SW_Push_Dual SW5
-U 1 1 5C3351EF
-P 1300 3250
-F 0 "SW5" H 1300 3535 50  0000 C CNN
-F 1 "SW_Push_Dual" H 1300 3444 50  0000 C CNN
-F 2 "Button_Switch_THT:Push E-Switch 6mm" H 1300 3450 50  0001 C CNN
-F 3 "" H 1300 3450 50  0001 C CNN
-	1    1300 3250
-	1    0    0    -1
-$EndComp
 Text GLabel 1700 3350 2    50   Input ~ 0
 SW_MODE_5
@@
 Wire Wire Line
 	1600 3350 1600 3450
-$Comp
-L Switch:SW_Push_Dual SW6
-U 1 1 5C340233
-P 1300 3850
-F 0 "SW6" H 1300 4135 50  0000 C CNN
-F 1 "SW_Push_Dual" H 1300 4044 50  0000 C CNN
-F 2 "Button_Switch_THT:Push E-Switch 6mm" H 1300 4050 50  0001 C CNN
-F 3 "" H 1300 4050 50  0001 C CNN
-	1    1300 3850
-	1    0    0    -1
-$EndComp
 Text GLabel 1700 3950 2    50   Input ~ 0
 SW_MODE_6
@@
 Wire Wire Line
 	5700 5800 5700 5700
+$Comp
+L Switch:SW_Push_4pin SW1
+U 1 1 5C24FD56
+P 1300 950
+F 0 "SW1" H 1300 1335 50  0000 C CNN
+F 1 "SW_Push_4pin" H 1300 1244 50  0000 C CNN
+F 2 "Button_Switch_THT:Push E-Switch 6mm" H 1300 950 50  0001 C CNN
+F 3 "" H 1300 950 50  0001 C CNN
+	1    1300 950
+	1    0    0    -1
+$EndComp
+$Comp
+L Switch:SW_Push_4pin SW2
+U 1 1 5C26992A
+P 1300 1550
+F 0 "SW2" H 1300 1935 50  0000 C CNN
+F 1 "SW_Push_4pin" H 1300 1844 50  0000 C CNN
+F 2 "Button_Switch_THT:Push E-Switch 6mm" H 1300 1550 50  0001 C CNN
+F 3 "" H 1300 1550 50  0001 C CNN
+	1    1300 1550
+	1    0    0    -1
+$EndComp
+$Comp
+L Switch:SW_Push_4pin SW4
+U 1 1 5C269BBD
+P 1300 2750
+F 0 "SW4" H 1300 3135 50  0000 C CNN
+F 1 "SW_Push_4pin" H 1300 3044 50  0000 C CNN
+F 2 "Button_Switch_THT:Push E-Switch 6mm" H 1300 2750 50  0001 C CNN
+F 3 "" H 1300 2750 50  0001 C CNN
+	1    1300 2750
+	1    0    0    -1
+$EndComp
+$Comp
+L Switch:SW_Push_4pin SW6
+U 1 1 5C282DFA
+P 1300 3950
+F 0 "SW6" H 1300 4335 50  0000 C CNN
+F 1 "SW_Push_4pin" H 1300 4244 50  0000 C CNN
+F 2 "Button_Switch_THT:Push E-Switch 6mm" H 1300 3950 50  0001 C CNN
+F 3 "" H 1300 3950 50  0001 C CNN
+	1    1300 3950
+	1    0    0    -1
+$EndComp
+$Comp
+L Switch:SW_Push_4pin SW5
+U 1 1 5C29C03C
+P 1300 3350
+F 0 "SW5" H 1300 3735 50  0000 C CNN
+F 1 "SW_Push_4pin" H 1300 3644 50  0000 C CNN
+F 2 "Button_Switch_THT:Push E-Switch 6mm" H 1300 3350 50  0001 C CNN
+F 3 "" H 1300 3350 50  0001 C CNN
+	1    1300 3350
+	1    0    0    -1
+$EndComp
+$Comp
+L Switch:SW_Push_4pin SW3
+U 1 1 5C2B527B
+P 1300 2150
+F 0 "SW3" H 1300 2535 50  0000 C CNN
+F 1 "SW_Push_4pin" H 1300 2444 50  0000 C CNN
+F 2 "Button_Switch_THT:Push E-Switch 6mm" H 1300 2150 50  0001 C CNN
+F 3 "" H 1300 2150 50  0001 C CNN
+	1    1300 2150
+	1    0    0    -1
+$EndComp
+$Comp
+L Mechanical:MountingHole MH?
+U 1 1 5C307B02
+P 10150 5450
+AR Path="/5BFAB137/5C307B02" Ref="MH?"  Part="1"
+AR Path="/5BFAD561/5C307B02" Ref="MH1"  Part="1"
+F 0 "MH1" H 10250 5496 50  0000 L CNN
+F 1 "MountingHole" H 10250 5405 50  0000 L CNN
+F 2 "MountingHole:MountingHole_3.2mm_M3" H 10150 5450 50  0001 C CNN
+F 3 "~" H 10150 5450 50  0001 C CNN
+	1    10150 5450
+	1    0    0    -1
+$EndComp
+$Comp
+L Mechanical:MountingHole MH?
+U 1 1 5C307B09
+P 10150 5700
+AR Path="/5BFAB137/5C307B09" Ref="MH?"  Part="1"
+AR Path="/5BFAD561/5C307B09" Ref="MH2"  Part="1"
+F 0 "MH2" V 10104 5800 50  0000 L CNN
+F 1 "MountingHole" V 10195 5800 50  0000 L CNN
+F 2 "MountingHole:MountingHole_3.2mm_M3" H 10150 5700 50  0001 C CNN
+F 3 "~" H 10150 5700 50  0001 C CNN
+	1    10150 5700
+	0    1    1    0
+$EndComp
+$Comp
+L Mechanical:MountingHole MH?
+U 1 1 5C307B10
+P 10150 5950
+AR Path="/5BFAB137/5C307B10" Ref="MH?"  Part="1"
+AR Path="/5BFAD561/5C307B10" Ref="MH3"  Part="1"
+F 0 "MH3" H 10250 5996 50  0000 L CNN
+F 1 "MountingHole" H 10250 5905 50  0000 L CNN
+F 2 "MountingHole:MountingHole_3.2mm_M3" H 10150 5950 50  0001 C CNN
+F 3 "~" H 10150 5950 50  0001 C CNN
+	1    10150 5950
+	1    0    0    -1
+$EndComp
 $EndSCHEMATC

Commit message: Fixed Component pinouts
Connections:
- wire segments 278 -> 279
Changed lines of the file:
@@
 	0    1    1    0
 $EndComp
-$Comp
-L power:Earth #PWR0115
-U 1 1 5C233BE0
-P 6600 1550
-F 0 "#PWR0115" H 6600 1300 50  0001 C CNN
-F 1 "Earth" H 6600 1400 50  0001 C CNN
-F 2 "" H 6600 1550 50  0001 C CNN
-F 3 "~" H 6600 1550 50  0001 C CNN
-	1    6600 1550
-	1    0    0    -1
-$EndComp
-Wire Wire Line
-	6600 1550 6600 1500
 Wire Wire Line
 	6600 1500 6650 1500
@@
 	0    1    1    0
 $EndComp
-$Comp
-L power:Earth #PWR0116
-U 1 1 5C233BFF
-P 7050 1550
-F 0 "#PWR0116" H 7050 1300 50  0001 C CNN
-F 1 "Earth" H 7050 1400 50  0001 C CNN
-F 2 "" H 7050 1550 50  0001 C CNN
-F 3 "~" H 7050 1550 50  0001 C CNN
-	1    7050 1550
-	1    0    0    -1
-$EndComp
-Wire Wire Line
-	7050 1550 7050 1500
 Wire Wire Line
 	7050 1500 7100 1500
@@
 	0    1    1    0
 $EndComp
-$Comp
-L power:Earth #PWR0117
-U 1 1 5C233C2C
-P 7500 1550
-F 0 "#PWR0117" H 7500 1300 50  0001 C CNN
-F 1 "Earth" H 7500 1400 50  0001 C CNN
-F 2 "" H 7500 1550 50  0001 C CNN
-F 3 "~" H 7500 1550 50  0001 C CNN
-	1    7500 1550
-	1    0    0    -1
-$EndComp
-Wire Wire Line
-	7500 1550 7500 1500
 Wire Wire Line
 	7500 1500 7550 1500
@@
 	0    1    1    0
 $EndComp
-$Comp
-L power:Earth #PWR0118
-U 1 1 5C233CBF
-P 7950 1550
-F 0 "#PWR0118" H 7950 1300 50  0001 C CNN
-F 1 "Earth" H 7950 1400 50  0001 C CNN
-F 2 "" H 7950 1550 50  0001 C CNN
-F 3 "~" H 7950 1550 50  0001 C CNN
-	1    7950 1550
-	1    0    0    -1
-$EndComp
-Wire Wire Line
-	7950 1550 7950 1500
 Wire Wire Line
 	7950 1500 8000 1500
@@
 	0    1    1    0
 $EndComp
-$Comp
-L power:Earth #PWR0119
-U 1 1 5C233D19
-P 8400 1550
-F 0 "#PWR0119" H 8400 1300 50  0001 C CNN
-F 1 "Earth" H 8400 1400 50  0001 C CNN
-F 2 "" H 8400 1550 50  0001 C CNN
-F 3 "~" H 8400 1550 50  0001 C CNN
-	1    8400 1550
-	1    0    0    -1
-$EndComp
-Wire Wire Line
-	8400 1550 8400 1500
 Wire Wire Line
 	8400 1500 8450 1500
 Wire Wire Line
-	8800 1200 8800 1500
-Wire Wire Line
 	8800 1500 8750 1500
 Wire Wire Line
 	6950 1500 7000 1500
 Wire Wire Line
-	7000 1500 7000 1200
-Connection ~ 7000 1200
-Wire Wire Line
-	7000 1200 7450 1200
-Wire Wire Line
 	7400 1500 7450 1500
 Wire Wire Line
-	7450 1500 7450 1200
-Connection ~ 7450 1200
-Wire Wire Line
-	7450 1200 7900 1200
-Wire Wire Line
 	7850 1500 7900 1500
 Wire Wire Line
-	7900 1500 7900 1200
-Connection ~ 7900 1200
-Wire Wire Line
-	7900 1200 8350 1200
-Wire Wire Line
 	6500 1500 6550 1500
 Wire Wire Line
-	6550 1500 6550 1200
-Wire Wire Line
-	6550 1200 7000 1200
-Wire Wire Line
 	8300 1500 8350 1500
-Wire Wire Line
-	8350 1500 8350 1200
-Connection ~ 8350 1200
-Wire Wire Line
-	8350 1200 8800 1200
 $Comp
 L 4xxx:4051 IC6
@@
 Wire Wire Line
 	1500 6350 1400 6350
-$Comp
-L power:Earth #PWR0114
-U 1 1 5C083E00
-P 6150 1550
-F 0 "#PWR0114" H 6150 1300 50  0001 C CNN
-F 1 "Earth" H 6150 1400 50  0001 C CNN
-F 2 "" H 6150 1550 50  0001 C CNN
-F 3 "~" H 6150 1550 50  0001 C CNN
-	1    6150 1550
-	1    0    0    -1
-$EndComp
-Wire Wire Line
-	6150 1550 6150 1500
 Wire Wire Line
 	6150 1500 6200 1500
@@
 Wire Wire Line
 	8800 1200 8800 1100
-Connection ~ 8800 1200
 Wire Wire Line
 	8250 3800 8250 3700
@@
 	1    0    0    -1
 $EndComp
+Wire Wire Line
+	6150 1200 6150 1500
+Wire Wire Line
+	6150 1200 6600 1200
+Wire Wire Line
+	6600 1500 6600 1200
+Connection ~ 6600 1200
+Wire Wire Line
+	6600 1200 7050 1200
+Wire Wire Line
+	7050 1500 7050 1200
+Connection ~ 7050 1200
+Wire Wire Line
+	7050 1200 7500 1200
+Wire Wire Line
+	7500 1500 7500 1200
+Connection ~ 7500 1200
+Wire Wire Line
+	7500 1200 7950 1200
+Wire Wire Line
+	7950 1500 7950 1200
+Connection ~ 7950 1200
+Wire Wire Line
+	7950 1200 8400 1200
+Wire Wire Line
+	8400 1500 8400 1200
+Connection ~ 8400 1200
+Wire Wire Line
+	8400 1200 8800 1200
+$Comp
+L power:Earth #PWR0115
+U 1 1 5D8C88F8
+P 6550 1550
+F 0 "#PWR0115" H 6550 1300 50  0001 C CNN
+F 1 "Earth" H 6550 1400 50  0001 C CNN
+F 2 "" H 6550 1550 50  0001 C CNN
+F 3 "~" H 6550 1550 50  0001 C CNN
+	1    6550 1550
+	1    0    0    -1
+$EndComp
+Wire Wire Line
+	6550 1550 6550 1500
+$Comp
+L power:Earth #PWR0116
+U 1 1 5D8E086D
+P 7000 1550
+F 0 "#PWR0116" H 7000 1300 50  0001 C CNN
+F 1 "Earth" H 7000 1400 50  0001 C CNN
+F 2 "" H 7000 1550 50  0001 C CNN
+F 3 "~" H 7000 1550 50  0001 C CNN
+	1    7000 1550
+	1    0    0    -1
+$EndComp
+Wire Wire Line
+	7000 1550 7000 1500
+$Comp
+L power:Earth #PWR0117
+U 1 1 5D8F8992
+P 7450 1550
+F 0 "#PWR0117" H 7450 1300 50  0001 C CNN
+F 1 "Earth" H 7450 1400 50  0001 C CNN
+F 2 "" H 7450 1550 50  0001 C CNN
+F 3 "~" H 7450 1550 50  0001 C CNN
+	1    7450 1550
+	1    0    0    -1
+$EndComp
+Wire Wire Line
+	7450 1550 7450 1500
+$Comp
+L power:Earth #PWR0118
+U 1 1 5D910C5B
+P 7900 1550
+F 0 "#PWR0118" H 7900 1300 50  0001 C CNN
+F 1 "Earth" H 7900 1400 50  0001 C CNN
+F 2 "" H 7900 1550 50  0001 C CNN
+F 3 "~" H 7900 1550 50  0001 C CNN
+	1    7900 1550
+	1    0    0    -1
+$EndComp
+Wire Wire Line
+	7900 1550 7900 1500
+$Comp
+L power:Earth #PWR0119
+U 1 1 5D9290B9
+P 8350 1550
+F 0 "#PWR0119" H 8350 1300 50  0001 C CNN
+F 1 "Earth" H 8350 1400 50  0001 C CNN
+F 2 "" H 8350 1550 50  0001 C CNN
+F 3 "~" H 8350 1550 50  0001 C CNN
+	1    8350 1550
+	1    0    0    -1
+$EndComp
+Wire Wire Line
+	8350 1550 8350 1500
+$Comp
+L power:Earth #PWR0221
+U 1 1 5D94169D
+P 8800 1550
+F 0 "#PWR0221" H 8800 1300 50  0001 C CNN
+F 1 "Earth" H 8800 1400 50  0001 C CNN
+F 2 "" H 8800 1550 50  0001 C CNN
+F 3 "~" H 8800 1550 50  0001 C CNN
+	1    8800 1550
+	1    0    0    -1
+$EndComp
+Wire Wire Line
+	8800 1550 8800 1500
 $EndSCHEMATC
