File: Power.sch (KiCad schematic (older format))
At the start: 22 parts, among them IC11 LM4040DBZ-2.5, IC2 R-78E3.3-0.5, IC7 LD2981ABU33

Commit message: Progress on routing tracks
Most of the power tracks are routed
Parts:
- C1, C10, C19, C2, C20, C21, C23, C25: footprint Capacitor_SMD:C_1206_3216Metric_Pad1.42x1.75mm_HandSolder -> Capacitor_SMD:C_1206_3216Metric
- C15, C17, C41: footprint Capacitor_SMD:C_0603_1608Metric_Pad1.05x0.95mm_HandSolder -> Capacitor_SMD:C_0805_2012Metric
- JP5: footprint Connector_PinHeader_2.54mm:PinHeader_2x05_P2.54mm_Vertical -> Connector_PinHeader_2.54mm:PinHeader_2x05_P2.54mm_Vertical_SMD
- L1, L4, L5, R33: footprint Resistor_SMD:R_0603_1608Metric_Pad1.05x0.95mm_HandSolder -> Resistor_SMD:R_0805_2012Metric
- L3: footprint Inductor_SMD:L_0805_2012Metric_Pad1.15x1.40mm_HandSolder -> Inductor_SMD:L_0805_2012Metric
Changed lines of the file:
@@
 F 0 "JP5" H 2700 2967 50  0000 C CNN
 F 1 "M05X2SMD" H 2700 2876 50  0000 C CNN
-F 2 "Connector_PinHeader_2.54mm:PinHeader_2x05_P2.54mm_Vertical" H 2650 2550 50  0001 C CNN
+F 2 "Connector_PinHeader_2.54mm:PinHeader_2x05_P2.54mm_Vertical_SMD" H 2650 2550 50  0001 C CNN
 F 3 "~" H 2650 2550 50  0001 C CNN
 	1    2650 2550
@@
 F 0 "L5" V 3426 2150 50  0000 C CNN
 F 1 "Ferrite_Bead" V 3517 2150 50  0000 C CNN
-F 2 "Resistor_SMD:R_0603_1608Metric_Pad1.05x0.95mm_HandSolder" V 3630 2150 50  0001 C CNN
+F 2 "Resistor_SMD:R_0805_2012Metric" V 3630 2150 50  0001 C CNN
 F 3 "~" H 3700 2150 50  0001 C CNN
 	1    3700 2150
@@
 F 0 "L1" V 3882 2950 50  0000 C CNN
 F 1 "Ferrite_Bead" V 3973 2950 50  0000 C CNN
-F 2 "Resistor_SMD:R_0603_1608Metric_Pad1.05x0.95mm_HandSolder" V 3630 2950 50  0001 C CNN
+F 2 "Resistor_SMD:R_0805_2012Metric" V 3630 2950 50  0001 C CNN
 F 3 "~" H 3700 2950 50  0001 C CNN
 	1    3700 2950
@@
 F 0 "C21" H 4215 2396 50  0000 L CNN
 F 1 "22u" H 4215 2305 50  0000 L CNN
-F 2 "Capacitor_SMD:C_1206_3216Metric_Pad1.42x1.75mm_HandSolder" H 4100 2350 50  0001 C CNN
+F 2 "Capacitor_SMD:C_1206_3216Metric" H 4100 2350 50  0001 C CNN
 F 3 "~" H 4100 2350 50  0001 C CNN
 	1    4100 2350
@@
 F 0 "C1" H 4215 2796 50  0000 L CNN
 F 1 "22u" H 4215 2705 50  0000 L CNN
-F 2 "Capacitor_SMD:C_1206_3216Metric_Pad1.42x1.75mm_HandSolder" H 4100 2750 50  0001 C CNN
+F 2 "Capacitor_SMD:C_1206_3216Metric" H 4100 2750 50  0001 C CNN
 F 3 "~" H 4100 2750 50  0001 C CNN
 	1    4100 2750
@@
 F 0 "C25" H 4615 2396 50  0000 L CNN
 F 1 "22u" H 4615 2305 50  0000 L CNN
-F 2 "Capacitor_SMD:C_1206_3216Metric_Pad1.42x1.75mm_HandSolder" H 4500 2350 50  0001 C CNN
+F 2 "Capacitor_SMD:C_1206_3216Metric" H 4500 2350 50  0001 C CNN
 F 3 "~" H 4500 2350 50  0001 C CNN
 	1    4500 2350
@@
 F 0 "C2" H 4615 2796 50  0000 L CNN
 F 1 "22u" H 4615 2705 50  0000 L CNN
-F 2 "Capacitor_SMD:C_1206_3216Metric_Pad1.42x1.75mm_HandSolder" H 4500 2750 50  0001 C CNN
+F 2 "Capacitor_SMD:C_1206_3216Metric" H 4500 2750 50  0001 C CNN
 F 3 "~" H 4500 2750 50  0001 C CNN
 	1    4500 2750
@@
 F 0 "R33" V 4795 2950 50  0000 C CNN
 F 1 "10k" V 4886 2950 50  0000 C CNN
-F 2 "Resistor_SMD:R_0603_1608Metric_Pad1.05x0.95mm_HandSolder" V 5040 2940 50  0001 C CNN
+F 2 "Resistor_SMD:R_0805_2012Metric" V 5040 2940 50  0001 C CNN
 F 3 "~" H 5000 2950 50  0001 C CNN
 	1    5000 2950
@@
 F 0 "C41" H 6315 3196 50  0000 L CNN
 F 1 "1u" H 6315 3105 50  0000 L CNN
-F 2 "Capacitor_SMD:C_0603_1608Metric_Pad1.05x0.95mm_HandSolder" H 6200 3150 50  0001 C CNN
+F 2 "Capacitor_SMD:C_0805_2012Metric" H 6200 3150 50  0001 C CNN
 F 3 "~" H 6200 3150 50  0001 C CNN
 	1    6200 3150
@@
 F 0 "L4" V 6963 2300 50  0000 C CNN
 F 1 "Ferrite_Bead_Small" V 7054 2300 50  0000 C CNN
-F 2 "Resistor_SMD:R_0603_1608Metric_Pad1.05x0.95mm_HandSolder" V 7130 2300 50  0001 C CNN
+F 2 "Resistor_SMD:R_0805_2012Metric" V 7130 2300 50  0001 C CNN
 F 3 "~" H 7200 2300 50  0001 C CNN
 	1    7200 2300
@@
 F 0 "C23" H 7515 2596 50  0000 L CNN
 F 1 "22u" H 7515 2505 50  0000 L CNN
-F 2 "Capacitor_SMD:C_1206_3216Metric_Pad1.42x1.75mm_HandSolder" H 7400 2550 50  0001 C CNN
+F 2 "Capacitor_SMD:C_1206_3216Metric" H 7400 2550 50  0001 C CNN
 F 3 "~" H 7400 2550 50  0001 C CNN
 	1    7400 2550
@@
 F 0 "C20" H 8515 2596 50  0000 L CNN
 F 1 "22u" H 8515 2505 50  0000 L CNN
-F 2 "Capacitor_SMD:C_1206_3216Metric_Pad1.42x1.75mm_HandSolder" H 8400 2550 50  0001 C CNN
+F 2 "Capacitor_SMD:C_1206_3216Metric" H 8400 2550 50  0001 C CNN
 F 3 "~" H 8400 2550 50  0001 C CNN
 	1    8400 2550
@@
 F 0 "C17" H 7315 1596 50  0000 L CNN
 F 1 "22u" H 7315 1505 50  0000 L CNN
-F 2 "Capacitor_SMD:C_0603_1608Metric_Pad1.05x0.95mm_HandSolder" H 7200 1550 50  0001 C CNN
+F 2 "Capacitor_SMD:C_0805_2012Metric" H 7200 1550 50  0001 C CNN
 F 3 "~" H 7200 1550 50  0001 C CNN
 	1    7200 1550
@@
 F 0 "C19" H 8215 1596 50  0000 L CNN
 F 1 "22u" H 8215 1505 50  0000 L CNN
-F 2 "Capacitor_SMD:C_1206_3216Metric_Pad1.42x1.75mm_HandSolder" H 8100 1550 50  0001 C CNN
+F 2 "Capacitor_SMD:C_1206_3216Metric" H 8100 1550 50  0001 C CNN
 F 3 "~" H 8100 1550 50  0001 C CNN
 	1    8100 1550
@@
 F 0 "C10" H 9215 1596 50  0000 L CNN
 F 1 "22u" H 9215 1505 50  0000 L CNN
-F 2 "Capacitor_SMD:C_1206_3216Metric_Pad1.42x1.75mm_HandSolder" H 9100 1550 50  0001 C CNN
+F 2 "Capacitor_SMD:C_1206_3216Metric" H 9100 1550 50  0001 C CNN
 F 3 "~" H 9100 1550 50  0001 C CNN
 	1    9100 1550
@@
 F 0 "C15" H 9615 1596 50  0000 L CNN
 F 1 "100n" H 9615 1505 50  0000 L CNN
-F 2 "Capacitor_SMD:C_0603_1608Metric_Pad1.05x0.95mm_HandSolder" H 9500 1550 50  0001 C CNN
+F 2 "Capacitor_SMD:C_0805_2012Metric" H 9500 1550 50  0001 C CNN
 F 3 "~" H 9500 1550 50  0001 C CNN
 	1    9500 1550
@@
 F 0 "L3" H 7650 1515 50  0000 C CNN
 F 1 "33u" H 7650 1424 50  0000 C CNN
-F 2 "Inductor_SMD:L_0805_2012Metric_Pad1.15x1.40mm_HandSolder" H 7650 1300 50  0001 C CNN
+F 2 "Inductor_SMD:L_0805_2012Metric" H 7650 1300 50  0001 C CNN
 F 3 "" H 7650 1300 50  0001 C CNN
 	1    7650 1300

Commit message: Added Mounting Holes
Parts:
- added MH4: MountingHole_Pad, Connector_PinHeader_1.00mm:PinHeader_1x01_P1.00mm_Vertical, symbol Mechanical:MountingHole_Pad
- renumbered D2 to D1, D1 to D2
Connections:
- wire segments 75 -> 76
Changed lines of the file:
@@
 	2350 2350 2850 2350
 $Comp
-L Device:D D2
+L Device:D D1
 U 1 1 5BFBF7D3
 P 3100 2750
-F 0 "D2" H 3100 2966 50  0000 C CNN
+F 0 "D1" H 3100 2966 50  0000 C CNN
 F 1 "D" H 3100 2875 50  0000 C CNN
 F 2 "Diode_SMD:D_SOD-123" H 3100 2750 50  0001 C CNN
@@
 $EndComp
 $Comp
-L Device:D D1
+L Device:D D2
 U 1 1 5BFBF834
 P 3100 2350
-F 0 "D1" H 3100 2134 50  0000 C CNN
+F 0 "D2" H 3100 2134 50  0000 C CNN
 F 1 "D" H 3100 2225 50  0000 C CNN
 F 2 "Diode_SMD:D_SOD-123" H 3100 2350 50  0001 C CNN
@@
 	9500 1300 9500 1200
 Connection ~ 9500 1300
+$Comp
+L Mechanical:MountingHole_Pad MH4
+U 1 1 5C2EB6D5
+P 3250 4800
+F 0 "MH4" H 3350 4851 50  0000 L CNN
+F 1 "MountingHole_Pad" H 3350 4760 50  0000 L CNN
+F 2 "Connector_PinHeader_1.00mm:PinHeader_1x01_P1.00mm_Vertical" H 3250 4800 50  0001 C CNN
+F 3 "~" H 3250 4800 50  0001 C CNN
+	1    3250 4800
+	1    0    0    -1
+$EndComp
+$Comp
+L power:Earth #PWR0220
+U 1 1 5C2EB7FD
+P 3250 5050
+F 0 "#PWR0220" H 3250 4800 50  0001 C CNN
+F 1 "Earth" H 3250 4900 50  0001 C CNN
+F 2 "" H 3250 5050 50  0001 C CNN
+F 3 "~" H 3250 5050 50  0001 C CNN
+	1    3250 5050
+	1    0    0    -1
+$EndComp
+Wire Wire Line
+	3250 4900 3250 5050
 $EndSCHEMATC

Commit message: Fixed Component pinouts
Changed lines of the file:
@@
 Wire Wire Line
 	3250 4900 3250 5050
+$Comp
+L power:PWR_FLAG #FLG0101
+U 1 1 5D9742E4
+P 2100 2650
+F 0 "#FLG0101" H 2100 2725 50  0001 C CNN
+F 1 "PWR_FLAG" H 2100 2824 50  0000 C CNN
+F 2 "" H 2100 2650 50  0001 C CNN
+F 3 "~" H 2100 2650 50  0001 C CNN
+	1    2100 2650
+	1    0    0    -1
+$EndComp
+Connection ~ 2100 2650
+$Comp
+L power:PWR_FLAG #FLG0102
+U 1 1 5D974352
+P 2850 2350
+F 0 "#FLG0102" H 2850 2425 50  0001 C CNN
+F 1 "PWR_FLAG" H 2850 2524 50  0000 C CNN
+F 2 "" H 2850 2350 50  0001 C CNN
+F 3 "~" H 2850 2350 50  0001 C CNN
+	1    2850 2350
+	1    0    0    -1
+$EndComp
+$Comp
+L power:PWR_FLAG #FLG0103
+U 1 1 5D9743C0
+P 2850 2750
+F 0 "#FLG0103" H 2850 2825 50  0001 C CNN
+F 1 "PWR_FLAG" H 2850 2923 50  0000 C CNN
+F 2 "" H 2850 2750 50  0001 C CNN
+F 3 "~" H 2850 2750 50  0001 C CNN
+	1    2850 2750
+	-1   0    0    1
+$EndComp
 $EndSCHEMATC
